File: A7585-test-board/A7585-test-board.sch (KiCad schematic (older format))
At the start: 38 parts, among them J1 Conn_01x04_Female, J100 Conn_Coaxial_Power, J2 Conn_01x20, J200 Conn_01x01_Female, J201 Conn_01x01_Female, J3 Conn_01x20, SW201 SW_SPDT, SW301 Rotary Encoder PCB, SW302 SW_Push_SPDT, SW303 SW_Push_SPDT, U100 MPM3610, U200 A7585D, U300 Pico, U301 LM4040LP-3

Commit message: Library-Reoganized
Parts:
- J1: footprint A7585-test-board:Connector_Strip -> A7585-footprints:Connector_Strip
- J200, J201: footprint A7585-test-board:Bannana_Jack_2pin -> A7585-footprints:Bannana_Jack_2pin
- RV301: footprint A7585-test-board:Potentiometer_Piher_T-16H_Single_Horizontal -> A7585-footprints:Potentiometer_Piher_T-16H_Single_Horizontal
- SW201: footprint A7585-test-board:SW_DIP_SPSTx01_Slide_9.78x4.72mm_W7.62mm_P2.54mm -> A7585-footprints:SW_DIP_SPSTx01_Slide_9.78x4.72mm_W7.62mm_P2.54mm
- SW302, SW303: footprint A7585-test-board:PUSH_BUTTON -> A7585-footprints:Push_Button
- U100: footprint A7585-test-board:MPM3610 -> A7585-footprints:MPM3610
- U200: footprint A7585-test-board:A7585D_Board -> A7585-footprints:A7585D_Board
- U300: footprint A7585-test-board:RPi_Pico_SMD_TH -> A7585-footprints:RPi_Pico_SMD_TH
Changed lines of the file:
@@
 F 0 "U200" H 5300 3215 50  0000 C CNN
 F 1 "A7585D" H 5300 3124 50  0000 C CNN
-F 2 "A7585-test-board:A7585D_Board" H 4750 3150 50  0001 C CNN
+F 2 "A7585-footprints:A7585D_Board" H 4750 3150 50  0001 C CNN
 F 3 "" H 4750 3150 50  0001 C CNN
 	1    5300 2350
@@
 F 0 "U300" H 5300 6315 50  0000 C CNN
 F 1 "Pico" H 5300 6224 50  0000 C CNN
-F 2 "A7585-test-board:RPi_Pico_SMD_TH" V 5300 5100 50  0001 C CNN
+F 2 "A7585-footprints:RPi_Pico_SMD_TH" V 5300 5100 50  0001 C CNN
 F 3 "" H 5300 5100 50  0001 C CNN
 	1    5300 5100
@@
 F 0 "SW201" H 1000 4000 50  0000 C CNN
 F 1 "SW_SPDT" H 950 3900 50  0000 C CNN
-F 2 "A7585-test-board:SW_DIP_SPSTx01_Slide_9.78x4.72mm_W7.62mm_P2.54mm" H 1150 3750 50  0001 C CNN
+F 2 "A7585-footprints:SW_DIP_SPSTx01_Slide_9.78x4.72mm_W7.62mm_P2.54mm" H 1150 3750 50  0001 C CNN
 F 3 "~" H 1150 3750 50  0001 C CNN
 	1    1150 3750
@@
 F 0 "U100" H 8858 1775 50  0000 C CNN
 F 1 "MPM3610" H 8858 1684 50  0000 C CNN
-F 2 "A7585-test-board:MPM3610" H 8800 1050 50  0001 C CNN
+F 2 "A7585-footprints:MPM3610" H 8800 1050 50  0001 C CNN
 F 3 "" H 8800 1050 50  0001 C CNN
 	1    8800 1400
@@
 F 0 "SW302" H 4150 4450 50  0000 C CNN
 F 1 "SW_Push_SPDT" H 3750 4644 50  0001 C CNN
-F 2 "A7585-test-board:PUSH_BUTTON" H 3750 4450 50  0001 C CNN
+F 2 "A7585-footprints:Push_Button" H 3750 4450 50  0001 C CNN
 F 3 "~" H 3750 4450 50  0001 C CNN
 	1    3750 4450
@@
 F 0 "SW303" H 3350 4550 50  0000 C CNN
 F 1 "SW_Push_SPDT" H 2950 4744 50  0001 C CNN
-F 2 "A7585-test-board:PUSH_BUTTON" H 2950 4550 50  0001 C CNN
+F 2 "A7585-footprints:Push_Button" H 2950 4550 50  0001 C CNN
 F 3 "~" H 2950 4550 50  0001 C CNN
 	1    2950 4550
@@
 F 0 "RV301" H 8132 5850 50  0000 R CNN
 F 1 "R_POT_US" H 8132 5805 50  0001 R CNN
-F 2 "A7585-test-board:Potentiometer_Piher_T-16H_Single_Horizontal" H 8200 5850 50  0001 C CNN
+F 2 "A7585-footprints:Potentiometer_Piher_T-16H_Single_Horizontal" H 8200 5850 50  0001 C CNN
 F 3 "~" H 8200 5850 50  0001 C CNN
 	1    8200 5850
@@
 F 0 "J1" V 3442 5312 50  0000 R CNN
 F 1 "Conn_01x04_Female" H 3578 5485 50  0001 L CNN
-F 2 "A7585-test-board:Connector_Strip" H 3550 5600 50  0001 C CNN
+F 2 "A7585-footprints:Connector_Strip" H 3550 5600 50  0001 C CNN
 F 3 "~" H 3550 5600 50  0001 C CNN
 	1    3550 5600
@@
 F 0 "J200" H 8878 2876 50  0000 L CNN
 F 1 "Conn_01x01_Female" H 8878 2785 50  0001 L CNN
-F 2 "A7585-test-board:Bannana_Jack_2pin" H 8850 2850 50  0001 C CNN
+F 2 "A7585-footprints:Bannana_Jack_2pin" H 8850 2850 50  0001 C CNN
 F 3 "~" H 8850 2850 50  0001 C CNN
 	1    8850 2850
@@
 F 0 "J201" H 8878 3026 50  0000 L CNN
 F 1 "Conn_01x01_Female" H 8878 2935 50  0001 L CNN
-F 2 "A7585-test-board:Bannana_Jack_2pin" H 8850 3000 50  0001 C CNN
+F 2 "A7585-footprints:Bannana_Jack_2pin" H 8850 3000 50  0001 C CNN
 F 3 "~" H 8850 3000 50  0001 C CNN
 	1    8850 3000

Commit message: Final Updates
Parts:
- added C112, C311, C313: 4.7 nF, Capacitor_SMD:C_1206_3216Metric, symbol Device:C
Connections:
- net GND: now also C112.2, C311.2, C313.2
- net at J2.11 (Pin_11), SW301.4 (Pin_4), U300.10 (GPIO7): now also C112.1
- net at J2.10 (Pin_10), U300.11 (GPIO8): now also SW301.3 (Pin_3), C313.1
- net at J2.12 (Pin_12), SW301.5 (Pin_5), U300.9 (GPIO6): now also C311.1
Changed lines of the file:
@@
 	2500 4950 2500 5350
 Wire Wire Line
-	2500 5350 1950 5350
+	2500 5350 2350 5350
 Connection ~ 4600 4950
 Wire Wire Line
-	4600 5050 2600 5050
+	4600 5050 2800 5050
 Wire Wire Line
 	2600 5050 2600 5450
@@
 	2600 5450 1950 5450
 Connection ~ 4600 5050
-Wire Wire Line
-	4550 5150 2700 5150
 Wire Wire Line
 	2700 5150 2700 5550
@@
 Wire Wire Line
 	8350 4650 9050 4650
+Wire Wire Line
+	2700 5150 3300 5150
+Connection ~ 4600 5150
+$Comp
+L Device:C C311
+U 1 1 6179C136
+P 2300 6650
+F 0 "C311" H 2415 6696 50  0000 L CNN
+F 1 "4.7 nF" H 2415 6605 50  0000 L CNN
+F 2 "Capacitor_SMD:C_1206_3216Metric" H 2338 6500 50  0001 C CNN
+F 3 "~" H 2300 6650 50  0001 C CNN
+	1    2300 6650
+	1    0    0    -1
+$EndComp
+$Comp
+L Device:C C112
+U 1 1 617A028B
+P 2750 6650
+F 0 "C112" H 2865 6696 50  0000 L CNN
+F 1 "4.7  nF" H 2865 6605 50  0000 L CNN
+F 2 "Capacitor_SMD:C_1206_3216Metric" H 2788 6500 50  0001 C CNN
+F 3 "~" H 2750 6650 50  0001 C CNN
+	1    2750 6650
+	1    0    0    -1
+$EndComp
+$Comp
+L Device:C C313
+U 1 1 617A687B
+P 3200 6650
+F 0 "C313" H 3315 6696 50  0000 L CNN
+F 1 "4.7 nF" H 3315 6605 50  0000 L CNN
+F 2 "Capacitor_SMD:C_1206_3216Metric" H 3238 6500 50  0001 C CNN
+F 3 "~" H 3200 6650 50  0001 C CNN
+	1    3200 6650
+	1    0    0    -1
+$EndComp
+Wire Wire Line
+	2350 5350 2350 6500
+Wire Wire Line
+	2350 6500 2300 6500
+Connection ~ 2350 5350
+Wire Wire Line
+	2350 5350 1950 5350
+Wire Wire Line
+	2800 5050 2800 6500
+Wire Wire Line
+	2800 6500 2750 6500
+Connection ~ 2800 5050
+Wire Wire Line
+	2800 5050 2600 5050
+Wire Wire Line
+	3300 5150 3300 6500
+Wire Wire Line
+	3300 6500 3200 6500
+Connection ~ 3300 5150
+Wire Wire Line
+	3300 5150 4600 5150
+$Comp
+L power:GND #PWR0139
+U 1 1 617C65CB
+P 2300 6800
+F 0 "#PWR0139" H 2300 6550 50  0001 C CNN
+F 1 "GND" H 2305 6627 50  0000 C CNN
+F 2 "" H 2300 6800 50  0001 C CNN
+F 3 "" H 2300 6800 50  0001 C CNN
+	1    2300 6800
+	1    0    0    -1
+$EndComp
+$Comp
+L power:GND #PWR0140
+U 1 1 617C6DA4
+P 2750 6800
+F 0 "#PWR0140" H 2750 6550 50  0001 C CNN
+F 1 "GND" H 2755 6627 50  0000 C CNN
+F 2 "" H 2750 6800 50  0001 C CNN
+F 3 "" H 2750 6800 50  0001 C CNN
+	1    2750 6800
+	1    0    0    -1
+$EndComp
+$Comp
+L power:GND #PWR0141
+U 1 1 617C70DC
+P 3200 6800
+F 0 "#PWR0141" H 3200 6550 50  0001 C CNN
+F 1 "GND" H 3205 6627 50  0000 C CNN
+F 2 "" H 3200 6800 50  0001 C CNN
+F 3 "" H 3200 6800 50  0001 C CNN
+	1    3200 6800
+	1    0    0    -1
+$EndComp
 $EndSCHEMATC
